File: Ki IP/System Circuit Low w Periph.kicad_sch (KiCad schematic)
At the start: 259 parts, among them J1 Barrel_Jack_Switch, J10 Conn_01x02, J11 Conn_01x02, J12 Screw_Terminal_01x02, J13 XT-90F-vert, J14 XT-90F-vert, J15 XT-90F-vert, J16 XT-90F-vert, J17 Screw_Terminal_01x02, J18 Screw_Terminal_01x02, J19 Screw_Terminal_01x02, J2 Conn_01x04, J20 Screw_Terminal_01x02, J21 Screw_Terminal_01x02, J22 Screw_Terminal_01x02, J23 Screw_Terminal_01x02, J24 Screw_Terminal_01x02, J25 Screw_Terminal_01x02, J26 Conn_01x02, J27 Conn_01x03, J28 Conn_01x03, J29 Conn_01x03, J3 Screw_Terminal_01x02, J30 Conn_01x03, J31 XT-90M-vert, J32 Conn_01x03, J33 Conn_01x03, J35 XT-90M-vert, J36 Conn_01x04, J37 XT-90F-vert, J38 XT-90M-vert, J39 Conn_01x02, J4 Screw_Terminal_01x02, J40 XT-90F-vert, J41 XT-90M-vert, J42 XT-90F-vert, J43 XT-90M-vert, J44 XT-90M-vert, J45 XT-90F-vert, J46 XT-90M-vert, J47 Conn_01x02, J48 XT-90F-vert, J49 XT-90F-vert, J5 Conn_02x02_Odd_Even, J50 XT-90M-vert, J51 XT-90M-vert, J52 XT-90F-vert, J53 XT-90M-vert, J54 Conn_01x02, J55 XT-90F-vert, J56 XT-90M-vert, J57 XT-90M-vert, J58 XT-90F-vert, J59 XT-90F-vert, J6 XT-90F-vert, J60 XT-90F-vert, J61 XT-90F-vert, J62 XT-90F-vert, J63 XT-90F-vert, J64 XT-90M-vert, J65 Conn_01x02, J66 XT-90F-vert, J67 XT-90M-vert, J68 Conn_01x03, J69 Conn_01x03, J7 Conn_02x03_Odd_Even, J70 XT-90F-vert, J71 XT-90F-vert, J72 XT-90F-vert, J73 Conn_01x03, J74 Conn_01x03, J75 Screw_Terminal_01x02, J8 Conn_02x03_Odd_Even, J9 Conn_01x02, K1 RT314A12, P1 Power Logger, P2 6s 17Ah 20C, P3 USB_C_Plug_USB2.0, Q1 HM2301B, Q3 IRF7403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

Commit message: add comments to describe pipeline
Parts:
- J13, J14, J15, J16, J37, J40, J42, J45, J48, J49, J52, J55, J58, J59, J6, J60, J61, J62, J63, J66, J70, J71, J72: value XT-90F-vert -> XT-90 F
- J31, J35, J38, J41, J43, J44, J46, J50, J51, J53, J56, J57, J64, J67: value XT-90M-vert -> XT-90 M
- renumbered U5 to BUCK1, U6 to BUCK2, U1 to BUCK3, U3 to BUCK4, J34 to E-STOP, U11 to ESC1, U12 to ESC2, U18 to ESC3, U24 to ESC4, U9 to MCU1, U4 to MCU2
Connections:
- net MAIN RETURN is gone; now on net In-Rush Limit: J35. (-)
- net MAIN SUPPLY is gone; now on net In-Rush Limit: J35. (-)
- net Earth: now also J35. (-)
- net Sig - DEPO BIN TILT: no longer ESC4. (S2), J65.2 (Pin_2)
- net Sig - EXC ASC/DSC: no longer ESC4. (S2), J65.1 (Pin_1)
- net Sig - EXCV TILT: no longer ESC3. (S2), J54.2 (Pin_2)
- net Sig - Ex Sprckt: no longer ESC3. (S2), J54.1 (Pin_1)
- net Sig - L1: no longer ESC1. (S2), J39.1 (Pin_1)
- net Sig - L2: no longer ESC1. (S2), J39.2 (Pin_2)
- net Sig - R1: no longer ESC2. (S2), J47.1 (Pin_1)
- net Sig - R2: no longer ESC2. (S2), J47.2 (Pin_2)
- net Sig - LF: now reaches ESC1. (S2)
- net Sig - LF: now also J39.1 (Pin_1); no longer J31. (-)
- net at J62. (-): now also J22.1 (Pin_1)
- net at J52. (-): now also ESC3. (S2)
- net Sig - Excv Tilt: now reaches ESC3. (S2)
- net Sig - Excv Tilt: now also J54.2 (Pin_2); no longer J52. (-)
- net Excv Asc/Dsc-: now reaches J64. (-)
- net at J60. (-): now also J18.1 (Pin_1)
- net at J42. (-): now also P1. (-); no longer J35. (-)
- net at J48. (-): now also J43. (-); no longer P2. (-)
- net at J37. (-): now also ESC1. (S2)
- net LF-: now reaches J38. (-)
- net at J49. (-): now also ESC2. (S2)
- net Sig - RF: now reaches ESC2. (S2)
- net Sig - RF: now also J47.1 (Pin_1); no longer J49. (-)
- net at J55. (-): now also ESC3. (S2)
- net at P1. (-): now also J43. (-); no longer J42. (-)
- net Depo Bin Tilt-: now reaches J67. (-)
- net Excv Tilt-: now reaches J56. (-)
- net at J6. (-): now also J12.1 (Pin_1)
- net at J58. (-): now also ESC4. (S2)
- net Sig - Excv Asc/Dsc: now reaches ESC4. (S2)
- net Sig - Excv Asc/Dsc: now also J65.1 (Pin_1); no longer J58. (-)
- net at J71. (-): now also J23.2 (Pin_2)
- net at J61. (-): now also U19.5 (IP-)
- net at J45. (-): now also ESC2. (S2)
- net at J40. (-): now also ESC1. (S2)
- net RB-: now reaches J50. (-)
- net RF-: now reaches J46. (-)
- net at J66. (-): no longer ESC4. (S2)
- net Excv Sprckt-: now reaches J53. (-)
- net LB-: now reaches J41. (-)
- new net: ESC1. (S2), J31. (-)
- new net: J13. (-), J14. (-), J15. (-), J16. (-), J75.2 (Pin_2)
- new net: ESC3. (S2), J52. (-)
- new net: J35. (-), J42. (-) (x2)
- new net: J48. (-), P2. (-)
- new net: ESC1. (S2), J37. (-)
- new net: ESC2. (S2), J49. (-)
- new net: ESC3. (S2), J55. (-)
- new net: ESC3. (S2), J51. (-)
- new net: J42. (-), P1. (-)
- new net: ESC4. (S2), J58. (-)
- new net: ESC4. (S2), J57. (-)
- new net: ESC2. (S2), J45. (-)
- new net: ESC2. (S2), J44. (-)
- new net: J43. (-), P1. (-)
- new net: ESC1. (S2), J40. (-)
- new net: J43. (-), J48. (-)
- new net: ESC4. (S2), J66. (-) (x2)
- new net Depo Bin Tilt+: J67. (-)
- new net Excv Asc/Dsc+: J64. (-)
- new net Excv Sprckt+: J53. (-)
- new net Excv Tilt+: J56. (-)
- new net LB+: J41. (-)
- new net LF+: J38. (-)
- new net RB+: J50. (-)
- new net RF+: J46. (-)
- new net Sig - Depo Bin Tilt: ESC4. (S2), J65.2 (Pin_2)
- new net Sig - Excv Sprckt: ESC3. (S2), J54.1 (Pin_1)
- new net Sig - LB: ESC1. (S2), J39.2 (Pin_2)
- new net Sig - RB: ESC2. (S2), J47.2 (Pin_2)
- now unconnected: J66. (-)
Other:
- moved on the sheet: E-STOP, J36, U10
